Commit message: Quad updated

File: defaultBody.urdf (robot description, URDF)
Before this commit: robot robot, 13 links, 12 joints
Links:
- removed link BackLeftLeg
- removed link BackRightLeg
- removed link FrontLeftLeg
- removed link FrontRightLeg
- removed link backLeftLowerLeg
- removed link backRightLowerLeg
- removed link frontLeftLowerLeg
- removed link frontRightLowerLeg
- removed link middleLeftLowerLeg
- removed link middleRightLowerLeg
- added link BackLeg, mass 1; collision box size=0.2 1 0.2; visual box size=0.2 1 0.2
- added link FrontLeg, mass 1; collision box size=0.2 1 0.2; visual box size=0.2 1 0.2
- added link LowerBackLeg, mass 1; collision box size=0.2 1 0.2; visual box size=0.2 1 0.2
- added link LowerFrontLeg, mass 1; collision box size=0.2 1 0.2; visual box size=0.2 1 0.2
- added link LowerLeftLeg, mass 1; collision box size=1 0.2 0.2; visual box size=1 0.2 0.2
- added link LowerRightLeg, mass 1; collision box size=1 0.2 0.2; visual box size=1 0.2 0.2
- link Torso: geometry collision box size=1 1 1; visual box size=1 1 1
Joints:
- removed joint BackLeftLeg_backLeftLowerLeg
- removed joint BackRightLeg_backRightLowerLeg
- removed joint FrontLeftLeg_frontLeftLowerLeg
- removed joint FrontRightLeg_frontRightLowerLeg
- removed joint MiddleLeftLeg_middleLeftLowerLeg
- removed joint MiddleRightLeg_middleRightLowerLeg
- removed joint Torso_BackLeftLeg
- removed joint Torso_BackRightLeg
- removed joint Torso_FrontLeftLeg
- removed joint Torso_FrontRightLeg
- added joint BackLeg_LowerBackLeg: type revolute, parent BackLeg, child LowerBackLeg, origin xyz=0 -1 0 rpy=0 0 0, axis 1 0 0, limit lower=-3.14159 upper=3.14159 effort=0.0 velocity=0.0
- added joint FrontLeg_LowerFrontLeg: type revolute, parent FrontLeg, child LowerFrontLeg, origin xyz=0 1 0 rpy=0 0 0, axis 1 0 0, limit lower=-3.14159 upper=3.14159 effort=0.0 velocity=0.0
- added joint MiddleLeftLeg_LowerLeftLeg: type revolute, parent MiddleLeftLeg, child LowerLeftLeg, origin xyz=-1 0 0 rpy=0 0 0, axis 0 1 0, limit lower=-3.14159 upper=3.14159 effort=0.0 velocity=0.0
- added joint MiddleRightLeg_LowerRightLeg: type revolute, parent MiddleRightLeg, child LowerRightLeg, origin xyz=1 0 0 rpy=0 0 0, axis 0 1 0, limit lower=-3.14159 upper=3.14159 effort=0.0 velocity=0.0
- added joint Torso_BackLeg: type revolute, parent Torso, child BackLeg, origin xyz=0 -0.5 1 rpy=0 0 0, axis 0 1 0, limit lower=-3.14159 upper=3.14159 effort=0.0 velocity=0.0
- added joint Torso_FrontLeg: type revolute, parent Torso, child FrontLeg, origin xyz=0 0.5 1 rpy=0 0 0, axis 0 1 0, limit lower=-3.14159 upper=3.14159 effort=0.0 velocity=0.0
- joint Torso_MiddleLeftLeg: axis 0 1 0 -> 0 0 1
- joint Torso_MiddleRightLeg: axis 0 1 0 -> 0 0 1
